File: snow/mk-ltk-02-pcb/mk-ltk-02-pcb.kicad_pcb (KiCad board)
At the start: 2 copper layers, 408.5 x 122.8 mm, 217 parts, among them M0 SW_Push, M1 SW_Push, U1 Teensy++2.0_(Arduino)

Commit message: add usb cutouts and ground plane
Parts:
- added REF**: USB_Type-C_cut-out, _Local_footprints:USB_Type-C_cut-out, F.Cu at (121.4, 84.5)
- added REF**: USB_Type-C_cut-out, _Local_footprints:USB_Type-C_cut-out, F.Cu at (402.4, 84.5)
- moved D87 16.8 mm to (392.3, 98.8), turned to 0 degrees
- moved D82 2.53 mm to (381.6, 85.1)
- moved D76 2.53 mm to (362.5, 85.1)
- moved D70 2.53 mm to (343.5, 85.1)
- moved D64 2.53 mm to (319.7, 85.1)
- moved D59 2.53 mm to (300.6, 85.1)
- moved D54 2.53 mm to (281.6, 85.1)
- moved D48 2.53 mm to (262.5, 85.1)
- moved D42 2.53 mm to (238.7, 85.1)
- moved D37 2.53 mm to (219.7, 85.1)
- moved D31 2.53 mm to (200.6, 85.1)
- moved D26 2.53 mm to (181.6, 85.1)
- moved D18 2.53 mm to (157.8, 85.1)
Routing:
- net (no net): track 0.00 -> 1220.3 mm, vias 0 -> 6
- net Net-(D100-Pad1): track 438.9 -> 492.6 mm, vias 0 -> 3
- net Net-(A-1-Pad1): track 451.8 -> 479.5 mm
- net Net-(A'1-Pad1): track 473.6 -> 498.8 mm
- net Net-(A-Backspace1-Pad1): track 504.7 -> 529.8 mm
- net Net-(M0-Pad1): track 517.2 -> 533.9 mm
- net Net-(D87-Pad2): track 11.9 -> 25.0 mm
- net Net-(M1-Pad1): track 536.4 -> 549.3 mm
- net Net-(D18-Pad2): track 11.9 -> 20.3 mm
- net Net-(A-Caps1-Pad1): track 175.3 -> 181.5 mm, vias 0 -> 1
- net Net-(A-H1-Pad1): track 330.3 -> 335.4 mm
- net Net-(D82-Pad2): track 11.9 -> 15.9 mm
- net Net-(D76-Pad2): track 11.9 -> 15.9 mm
- net Net-(D70-Pad2): track 11.9 -> 15.9 mm
- net Net-(D64-Pad2): track 11.9 -> 15.9 mm
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- added copper zone on B.Cu, net Net-(U1-Pad33)
- added copper zone on F.Cu, net Net-(U1-Pad33)
Other:
- outline, holes or cut-outs redrawn
